Commit message: feat: IV2023 demo
Signed-off-by: Amadeusz Szymko <amadeusz.szymko@put.poznan.pl>

File: f1tenth_vehicle_description/urdf/vehicle.xacro (robot description, xacro)
@@ -6,9 +6,15 @@
   <link name="base_link">
     <visual>
-      <origin xyz="${vehicle_info['/**']['ros__parameters']['wheel_base']/2.0} 0 -${vehicle_info['/**']['ros__parameters']['wheel_radius']}" rpy="0 0 0"/>
+      <origin xyz="0.15371 0 -${vehicle_info['/**']['ros__parameters']['wheel_radius']}" rpy="0 0 ${pi/2.0}"/>
       <geometry>
-        <mesh filename="package://f1tenth_vehicle_description/mesh/f1tenth.dae" scale="1 1 1"/>
+        <mesh filename="package://f1tenth_vehicle_description/mesh/F1TenthVehicle.dae" scale="1 1 1"/>
       </geometry>
     </visual>
   </link>
+  <!-- <joint name="base_footprint_joint" type="fixed">
+    <origin xyz="0 0 -${vehicle_info['/**']['ros__parameters']['wheel_radius']}" rpy="0 0 0"/>
+    <parent link="base_link"/>
+    <child link="base_footprint"/>
+  </joint>
+  <link name="base_footprint"/> -->
 </robot>
